File: nand.kicad_sch (KiCad schematic)
At the start: 3 parts, among them U14 MT29F8G08ABACA

Commit message: add pullup to NAND R/B# as per ONFI 1.0 spec
Parts:
- added R13: 4.7k, Resistor_SMD:R_0402_1005Metric, symbol Device:R_Small
Connections:
- net +3V3: now also R13.1
- net R/~{B}: now also R13.2
Changed lines of the file:
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@@
+	)
+	(junction
+		(at 149.86 115.57)
+		(diameter 0)
+		(color 0 0 0 0)
 	)
 	(junction
@@
 	(wire
 		(pts
-			(xy 124.46 115.57) (xy 160.02 115.57)
+			(xy 124.46 115.57) (xy 149.86 115.57)
 		)
 		(stroke
@@
 	(wire
 		(pts
+			(xy 149.86 105.41) (xy 149.86 106.68)
+		)
+		(stroke
+			(width 0)
+			(type default)
+		)
+	)
+	(wire
+		(pts
 			(xy 176.53 93.98) (xy 176.53 96.52)
 		)
@@
 		)
 	)
+	(wire
+		(pts
+			(xy 149.86 111.76) (xy 149.86 115.57)
+		)
+		(stroke
+			(width 0)
+			(type default)
+		)
+	)
 	(bus
 		(pts
 			(xy 154.94 128.27) (xy 154.94 130.81)
+		)
+		(stroke
+			(width 0)
+			(type default)
+		)
+	)
+	(wire
+		(pts
+			(xy 149.86 115.57) (xy 160.02 115.57)
 		)
 		(stroke
@@
 					(unit 1)
 				)
+			)
+		)
+	)
+	(symbol
+		(lib_id "power:+3V3")
+		(at 149.86 105.41 0)
+		(unit 1)
+		(exclude_from_sim no)
+		(in_bom yes)
+		(on_board yes)
+		(dnp no)
+		(fields_autoplaced yes)
+		(property "Reference" "#PWR0153"
+			(at 149.86 109.22 0)
+			(effects
+				(font
+					(size 1.27 1.27)
+				)
+				(hide yes)
+			)
+		)
+		(property "Value" "+3V3"
+			(at 149.86 100.33 0)
+			(effects
+				(font
+					(size 1.27 1.27)
+				)
+			)
+		)
+		(property "Footprint" ""
+			(at 149.86 105.41 0)
+			(effects
+				(font
+					(size 1.27 1.27)
+				)
+				(hide yes)
+			)
+		)
+		(property "Datasheet" ""
+			(at 149.86 105.41 0)
+			(effects
+				(font
+					(size 1.27 1.27)
+				)
+				(hide yes)
+			)
+		)
+		(property "Description" "Power symbol creates a global label with name \"+3V3\""
+			(at 149.86 105.41 0)
+			(effects
+				(font
+					(size 1.27 1.27)
+				)
+				(hide yes)
+			)
+		)
+		(pin "1"
+		)
+		(instances
+			(project "ns32k"
+				(path "/54787df0-1b8c-465f-acae-f55ec7f02da3/bf4bb805-a9c2-47a8-9dba-461cccb7b358"
+					(reference "#PWR0153")
+					(unit 1)
+				)
+			)
+		)
+	)
+	(symbol
+		(lib_id "Device:R_Small")
+		(at 149.86 109.22 0)
+		(unit 1)
+		(exclude_from_sim no)
+		(in_bom yes)
+		(on_board yes)
+		(dnp no)
+		(fields_autoplaced yes)
+		(property "Reference" "R13"
+			(at 152.4 107.9499 0)
+			(effects
+				(font
+					(size 1.27 1.27)
+				)
+				(justify left)
+			)
+		)
+		(property "Value" "4.7k"
+			(at 152.4 110.4899 0)
+			(effects
+				(font
+					(size 1.27 1.27)
+				)
+				(justify left)
+			)
+		)
+		(property "Footprint" "Resistor_SMD:R_0402_1005Metric"
+			(at 149.86 109.22 0)
+			(effects
+				(font
+					(size 1.27 1.27)
+				)
+				(hide yes)
+			)
+		)
+		(property "Datasheet" "~"
+			(at 149.86 109.22 0)
+			(effects
+				(font
+					(size 1.27 1.27)
+				)
+				(hide yes)
+			)
+		)
+		(property "Description" "Resistor, small symbol"
+			(at 149.86 109.22 0)
+			(effects
+				(font
+					(size 1.27 1.27)
+				)
+				(hide yes)
+			)
+		)
+		(pin "1"
+		)
+		(pin "2"
+		)
+		(instances
+			(project "ns32k"
+				(path "/54787df0-1b8c-465f-acae-f55ec7f02da3/bf4bb805-a9c2-47a8-9dba-461cccb7b358"
+					(reference "R13")
+					(unit 1)
+				)

Commit message: fix address decoding
Parts:
- C28, C30: LCSC (none) -> C466613
- R13: LCSC (none) -> C380746
- U14: LCSC (none) -> C400999
Changed lines of the file:
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@@
 	(title_block
 		(title "NS32016 Toy PCB")
-		(date "2024-08-01")
+		(date "2024-08-10")
 		(rev "Rev 4")
 		(comment 1 "bson@rockgarden.net")
@@
 			)
 		)
+		(property "LCSC" "C400999"
+			(at 180.34 140.97 0)
+			(effects
+				(font
+					(size 1.27 1.27)
+				)
+				(hide yes)
+			)
+		)
 		(pin "10"
 		)
@@
 		)
 		(property "Description" "Resistor, small symbol"
+			(at 149.86 109.22 0)
+			(effects
+				(font
+					(size 1.27 1.27)
+				)
+				(hide yes)
+			)
+		)
+		(property "LCSC" "C380746"
 			(at 149.86 109.22 0)
 			(effects
@@
 			)
 		)
+		(property "LCSC" "C466613"
+			(at 187.96 101.6 0)
+			(effects
+				(font
+					(size 1.27 1.27)
+				)
+				(hide yes)
+			)
+		)
 		(pin "1"
 		)
@@
 			(at 172.72 101.6 0)
 			(effects
+				(font
+					(size 1.27 1.27)
+				)
+				(hide yes)
+			)
+		)
+		(property "LCSC" "C466613"
+			(at 172.72 101.6 0)
+			(effects

Commit message: various changes, add LCSC part #s
Parts:
- C28, C30: LCSC C466613 -> C3012376
- R13: LCSC C380746 -> C25940
Changed lines of the file:
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@@
 			)
 		)
-		(property "LCSC" "C380746"
+		(property "LCSC" "C25940"
 			(at 149.86 109.22 0)
 			(effects
@@
 			)
 		)
-		(property "LCSC" "C466613"
+		(property "LCSC" "C3012376"
 			(at 187.96 101.6 0)
 			(effects
@@
 			)
 		)
-		(property "LCSC" "C466613"
-			(at 172.72 101.6 0)
-			(effects
+		(property "LCSC" "C3012376"
+			(at 172.72 101.6 0)
+			(effects

Commit message: fix a few bugs
Other:
- title: NS32016 Toy PCB -> Toy32k
Changed lines of the file:
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@@
 	(paper "A3")
 	(title_block
-		(title "NS32016 Toy PCB")
-		(date "2024-08-10")
-		(rev "Rev 4")
+		(title "Toy32k")
+		(date "2024-08-16")
+		(rev "Rev 5")
 		(comment 1 "bson@rockgarden.net")
 		(comment 2 "Jan Brittenson")
